File: BAVGext.kicad_pcb (KiCad board)
At the start: 2 copper layers, 18 x 15 mm, 4 parts, among them J1 Conn_01x04, J2 Conn_01x04, J3 Conn_01x02, J4 Conn_01x02

Commit message: replace files
Parts:
- added R1: 120, Resistor_THT:R_Axial_DIN0207_L6.3mm_D2.5mm_P2.54mm_Vertical, F.Cu at (1.50, 13.2)
- J4: footprint Connector_PinSocket_2.54mm:PinSocket_1x02_P2.54mm_Vertical -> Connector_JST:JST_XH_B2B-XH-A_1x02_P2.50mm_Vertical
- moved J4 1.91 mm to (6.40, 11.5)
- moved J3 1.88 mm to (13.9, 11.6)
Routing:
- net /B: track 23.2 -> 17.9 mm
- net /V: track 21.0 -> 26.0 mm
- net /G: track 31.9 -> 34.7 mm
- net /A: track 21.4 -> 23.3 mm
- added copper zone on B.Cu, net /G
- added copper zone on F.Cu, net /G
Other:
- board text added: "120"
