File: BAVGext.kicad_sch (KiCad schematic)
At the start: 4 parts, among them J1 Conn_01x04, J2 Conn_01x04, J3 Conn_01x02, J4 Conn_01x02

Commit message: replace files
Parts:
- added R1: 120, Resistor_THT:R_Axial_DIN0207_L6.3mm_D2.5mm_P2.54mm_Vertical, symbol Device:R
- J4: footprint Connector_PinSocket_2.54mm:PinSocket_1x02_P2.54mm_Vertical -> Connector_JST:JST_XH_B2B-XH-A_1x02_P2.50mm_Vertical
Connections:
- net A: now also R1.2
- net B: now also R1.1
Changed lines of the file:
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@@
 (kicad_sch (version 20211123) (generator eeschema)
   (paper "A4")
+  (junction (at 72.39 50.8) (diameter 0) (color 0 0 0 0)
+  )
+  (junction (at 80.01 53.34) (diameter 0.0254) (color 0 0 0 0)
+  )
   (junction (at 76.2 68.58) (diameter 0) (color 0 0 0 0)
   )
@@
   )
   (wire (pts (xy 64.77 55.88) (xy 80.01 55.88))
+    (stroke (width 0) (type default) (color 0 0 0 0))
+  )
+  (wire (pts (xy 72.39 46.99) (xy 72.39 50.8))
     (stroke (width 0) (type default) (color 0 0 0 0))
   )
@@
     (stroke (width 0) (type default) (color 0 0 0 0))
   )
-  (wire (pts (xy 64.77 50.8) (xy 82.55 50.8))
+  (wire (pts (xy 64.77 50.8) (xy 72.39 50.8))
     (stroke (width 0) (type default) (color 0 0 0 0))
   )
@@
     (stroke (width 0) (type default) (color 0 0 0 0))
   )
-  (wire (pts (xy 64.77 53.34) (xy 82.55 53.34))
+  (wire (pts (xy 64.77 53.34) (xy 80.01 53.34))
+    (stroke (width 0) (type default) (color 0 0 0 0))
+  )
+  (wire (pts (xy 80.01 46.99) (xy 80.01 53.34))
+    (stroke (width 0) (type default) (color 0 0 0 0))
+  )
+  (wire (pts (xy 72.39 50.8) (xy 82.55 50.8))
+    (stroke (width 0) (type default) (color 0 0 0 0))
+  )
+  (wire (pts (xy 80.01 53.34) (xy 82.55 53.34))
     (stroke (width 0) (type default) (color 0 0 0 0))
   )
@@
       (effects (font (size 1.27 1.27)) (justify left))
     )
-    (property "Footprint" "Connector_PinSocket_2.54mm:PinSocket_1x02_P2.54mm_Vertical" (id 2) (at 87.63 72.39 0)
+    (property "Footprint" "Connector_JST:JST_XH_B2B-XH-A_1x02_P2.50mm_Vertical" (id 2) (at 87.63 72.39 0)
       (effects (font (size 1.27 1.27)) hide)
     )
     (property "Datasheet" "~" (id 3) (at 87.63 72.39 0)
+      (effects (font (size 1.27 1.27)) hide)
+    )
+    (pin "1")
+    (pin "2")
+  )
+  (symbol (lib_id "Device:R") (at 76.2 46.99 90) (unit 1)
+    (in_bom yes) (on_board yes) (fields_autoplaced)
+    (property "Reference" "R1" (id 0) (at 76.2 42.0075 90))
+    (property "Value" "120" (id 1) (at 76.2 44.7826 90))
+    (property "Footprint" "Resistor_THT:R_Axial_DIN0207_L6.3mm_D2.5mm_P2.54mm_Vertical" (id 2) (at 76.2 48.768 90)
+      (effects (font (size 1.27 1.27)) hide)
+    )
+    (property "Datasheet" "~" (id 3) (at 76.2 46.99 0)
       (effects (font (size 1.27 1.27)) hide)
     )
@@
     )
     (path "/f508a62c-3c21-46de-b321-51b8800cff11"
-      (reference "J4") (unit 1) (value "Conn_01x02") (footprint "Connector_PinSocket_2.54mm:PinSocket_1x02_P2.54mm_Vertical")
+      (reference "J4") (unit 1) (value "Conn_01x02") (footprint "Connector_JST:JST_XH_B2B-XH-A_1x02_P2.50mm_Vertical")
+    )
+    (path "/fd146ca2-8fb8-4c71-9277-84f69bc5d3fc"
+      (reference "R1") (unit 1) (value "120") (footprint "Resistor_THT:R_Axial_DIN0207_L6.3mm_D2.5mm_P2.54mm_Vertical")
     )
   )
